File: neuron_sig_gen.sch (EAGLE design)
At the start: 112 parts, among them IC1 AD8684RU, IC2 AD8684RU, IC3 ADA4692-2R, IC4 ADA4692-2R, SW1 B3U-1000P, U1 TPS72301DBVRSOT-23-5, U2 TLV703, X1 ABM3B-16.000MHZ-B2-T, X2 9HT10-32.768KDZF-T

Commit message: added new version with controller
Parts:
- removed BOOT0, BOOT1, BOOT2: (no value), pinhead:PINHD-1X3
- removed C14: 1uF, rcl:C-EUC0603
- removed C15, C16, C17, C20, C22, C23, C29: 100n, rcl:C-EUC0603K
- removed C19, C21: 2.2 u, rcl:C-EUC0603K
- removed C25, C26: 18p, rcl:C-EUC0603K
- removed C27, C28: 12.5p, rcl:C-EUC0603K
- removed ICA: AD5270MSOP10, untitled:AD5270MSOP10
- removed PB12, PB13, PB14, PB15, URXL, UTXL: LEDCHIPLED_0805, audio amplifier example:LEDCHIPLED_0805
- removed R10, R11, R12, R13, R14, R15, R16, R17, R18, R19, R20, R21, R22, R23, R24, R25, R26, R27, R28, R29, R30, R31, R32, R33, R34, R35, R36, R37, R38, R39, R40, R9: 10k, rcl:R-EU_R0603
- removed R41, R42, R47, R48, R49, R50: 180R, rcl:R-EU_R0603
- removed R51, R52: 10K, rcl:R-EU_R0603
- removed SW1: B3U-1000P, Switch:B3U-1000P
- removed SWD: B6B-ZR, jst:B6B-ZR
- removed U$1: STM32F405RGT6, SparkFun-IC-Microcontroller:STM32F405RG
- removed X1: ABM3B-16.000MHZ-B2-T, Crystals:ABM3B-16.000MHZ-B2-T
- removed X2: 9HT10-32.768KDZF-T, Crystals:9HT10-32.768KDZF-T
- added JP4: (no value), pinhead:PINHD-1X6
- IC1, IC2: value AD8684RU -> 74HC595D; device linear:AD8684RU -> 74xx-eu:74HC595D
Connections:
- removed net +3V3: BOOT0.3, BOOT1.3, C11.2, C15.2, C16.2, C17.2, C20.2, C22.2, C23.2, JP1.1, SWD.4, U$1.VBAT, U$1.VDD1, U$1.VDD2, U$1.VDD3, U$1.VDD4, U$1.VDDA, U2.EN, U2.IN
- removed net AQA: IC1A.OUT, ICA.A, R12.1
- removed net BOOT0: R51.2, U$1.BOOT0
- removed net BOOT1: R52.2, U$1.PB2-BOOT1
- removed net CS: U$1.PD2/SDIO_CMD
- removed net CSPOW: ICPOW.NCS
- removed net DAC1: U$1.PA4/SPI1_NSS
- removed net LED1: PB12.A, U$1.PB12/I2S2_WS
- removed net LED2: PB13.A, U$1.PB13/I2S2_CK
- removed net LED3: PB14.A, U$1.PB14/I2S2_XD
- removed net LED4: PB15.A, U$1.PB15/I2S2_SD
- removed net N$13: C14.2, ICA.CAP
- removed net N$15: IC1A.-IN, R10.1, R11.1
- removed net N$16: IC1B.+IN, R13.1, R16.2
- removed net N$18: IC1C.-IN, R18.1, R19.1
- removed net N$19: IC1C.+IN, R17.1, R20.2
- removed net N$21: IC1A.+IN, R12.2, R9.1
- removed net N$22: IC1D.-IN, R22.1, R23.1
- removed net N$23: IC1D.+IN, R21.1, R24.2
- removed net N$24: IC2A.-IN, R26.1, R27.1
- removed net N$25: IC2A.+IN, R25.1, R28.2
- removed net N$26: IC1B.-IN, R14.1, R15.1
- removed net N$27: IC2B.-IN, R30.1, R31.1
- removed net N$28: IC2B.+IN, R29.1, R32.2
- removed net N$29: IC2C.-IN, R34.1, R35.1
- removed net N$30: IC2C.+IN, R33.1, R36.2
- removed net N$31: IC2D.-IN, R38.1, R39.1
- removed net N$32: IC2D.+IN, R37.1, R40.2
- removed net N$33: C19.2, U$1.VCAP1
- removed net N$34: IC1B.OUT, R16.1
- removed net N$35: IC1C.OUT, R20.1
- removed net N$36: IC1D.OUT, R24.1
- removed net N$37: C21.2, U$1.VCAP2
- removed net N$38: IC2B.OUT, R32.1
- removed net N$39: IC2C.OUT, R36.1
- removed net N$40: IC2D.OUT, R40.1
- removed net N$41: R41.2, UTXL.C
- removed net N$42: R42.2, URXL.C
- removed net N$47: PB12.C, R47.2
- removed net N$48: PB13.C, R48.2
- removed net N$49: PB14.C, R49.2
- removed net N$50: PB15.C, R50.2
- removed net N$51: BOOT0.2, R51.1
- removed net N$52: BOOT1.2, R52.1
- removed net NRST: C29.2, SW1.2, SWD.1, U$1.NRST
- removed net Q1: R9.2
- removed net Q10: R26.2
- removed net Q11: R29.2
- removed net Q12: R30.2
- removed net Q13: R33.2
- removed net Q14: R34.2
- removed net Q15: R37.2
- removed net Q16: R38.2
- removed net Q2: R10.2
- removed net Q3: R13.2
- removed net Q4: R14.2
- removed net Q5: R17.2
- removed net Q6: R18.2
- removed net Q7: R21.2
- removed net Q8: R22.2
- removed net Q9: R25.2
- removed net RCC1: C26.1, U$1.PH0, X1.1
- removed net RCC2: C25.2, U$1.PH1, X1.3
- removed net RTC1: C27.1, U$1.PC14, X2.2
- removed net RTC2: C28.2, U$1.PC15, X2.1
- removed net SWCLK: SWD.2, U$1.PA14/JTCK
- removed net SWDIO: SWD.3, U$1.PA13/JTMS
- removed net URX: U$1.PA10/UART1_RX, URXL.A
- removed net UTX: U$1.PA9/UART1_TX, UTXL.A
- new net +5V: C11.2, JP1.1, U2.EN, U2.IN
- new net CS_CS: IC2A.RCK, JP4.2
- new net CS_IN: IC1A.RCK, JP4.1
- net +2V5: now also IC1A.SCL, IC1P.VCC, IC2A.SCL, IC2P.VCC; no longer IC1P.V+, IC2P.V+, ICA.VDD
- net -2V5: no longer IC1P.V-, IC2P.V-, ICA.VSS
- net AQB: now also IC1A.QB
- net AQC: now also IC1A.QC
- net AQD: now also IC1A.QD
- net AQE: now also IC1A.QE; no longer IC2A.OUT, R28.1
- net AQF: now also IC1A.QF
- net AQG: now also IC1A.QG
- net AQH: now also IC1A.QH
- net CSA: now also IC2A.QA, ICPOW.NCS; no longer ICA.NSYNC
- net CSB: now also IC2A.QB
- net CSC: now also IC2A.QC
- net CSD: now also IC2A.QD
- net CSE: now also IC2A.QE
- net CSF: now also IC2A.QF
- net CSG: now also IC2A.QG
- net CSH: now also IC2A.QH
- net GND: now also IC1A.G, IC1P.GND, IC2A.G, IC2P.GND, JP4.6; no longer BOOT0.1, BOOT1.1, BOOT2.1, C14.1, C15.1, C16.1, C17.1, C19.1, C20.1, C21.1, C22.1, C23.1, C25.1, C26.2, C27.2, C28.1, C29.1, ICA.GND, R11.2, R15.2, R19.2, R23.2, R27.2, R31.2, R35.2, R39.2, R41.1, R42.1, R47.1, R48.1, R49.1, R50.1, SW1.1, SWD.5, SWD.6, U$1.VSS1, U$1.VSS2, U$1.VSSA, X1.2, X1.4
- net MISO: now also JP4.3; no longer ICA.SDO, U$1.PC11/SDIO_D3
- net MOSI: now also IC1A.SER, IC2A.SER, JP4.4; no longer ICA.DIN, U$1.PC12/SDIO_CLK
- net SCLK: now also IC1A.SCK, IC2A.SCK, JP4.5; no longer ICA.SCLK, U$1.PC10/SDIO_D2
- net W: no longer ICA.W
Other:
- moved on the sheet: C1, C2, C3, C4, C5, C6, C7, IC3P, IC4P, ICB, ICC, ICD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
