File: neuron.brd (EAGLE design)
At the start: 40.6 x 48.3 mm, 44 parts, among them IC1 74HC595D, IC2 74HC595D, IC3 ADA4692-2R, IC4 ADA4692-2R, U1 TPS72301DBVRSOT-23-5, U2 TLV703

Commit message: added some measurements
Parts:
- moved LEDOUT 2.25 mm to (16.1, 45.7)
- moved JP2 1.65 mm to (20.3, 45.7)
- moved JP1 0.92 mm to (2.54, 20.3)
- moved R8 0.90 mm to (15.9, 42.4)
- moved JP4 0.28 mm to (24.1, 5.08)
Routing:
- net N$12: track 1.94 -> 4.43 mm
- net OUT: track 12.1 -> 10.7 mm
- net SCLK: track 106.9 -> 105.8 mm
- net -5V: track 10.6 -> 11.4 mm

Commit message: added new version with controller
Parts:
- removed JP4: (no value), pinhead:1X06
- added BOOT0, BOOT1, BOOT2: (no value), pinhead:1X03
- added C14: 1uF, rcl:C0603
- added C15, C16, C17, C20, C22, C23, C29: 100n, rcl:C0603K
- added C19, C21: 2.2 u, rcl:C0603K
- added C25, C26: 18p, rcl:C0603K
- added C27, C28: 12.5p, rcl:C0603K
- added ICA: AD5270MSOP10, untitled:MSOP10
- added PB12, PB13, PB14, PB15, URXL, UTXL: LEDCHIPLED_0805, audio amplifier example:CHIPLED_0805
- added R10, R11, R12, R13, R14, R15, R16, R17, R18, R19, R20, R21, R22, R23, R24, R25, R26, R27, R28, R29, R30, R31, R32, R33, R34, R35, R36, R37, R38, R39, R40, R9: 10k, rcl:R0603
- added R41, R42, R47, R48, R49, R50: 180R, rcl:R0603
- added R51, R52: 10K, rcl:R0603
- added SW1: B3U-1000P, Switch:B3U-1000P
- added SWD: B6B-ZR, jst:B6B-ZR
- added U$1: STM32F405RGT6, SparkFun-IC-Microcontroller:TQFP64
- added X1: ABM3B-16.000MHZ-B2-T, Crystals:ABM3B-16.000MHZ-B2-T
- added X2: 9HT10-32.768KDZF-T, Crystals:9HT10-32.768KDZF-T
- IC1, IC2: value 74HC595D -> AD8684RU; device 74xx-eu:SO16 -> linear:TSSOP14
- moved R4 35.0 mm to (-22.0, -0.13), turned to 180 degrees
- moved C11 31.2 mm to (-26.5, 31.8)
- moved C12 31.2 mm to (-18.9, 31.6)
- moved LED+2.5 31.2 mm to (-19.9, 34.4)
- moved R5 31.2 mm to (-24.8, 34.4)
- moved U2 31.2 mm to (-23.4, 31.6)
- moved LED-2.5 30.8 mm to (-21.7, 3.05), turned to 270 degrees
- moved C8 30.8 mm to (-21.7, 4.95), turned to 0 degrees
- moved C10 30.0 mm to (-24.6, 6.86), turned to 90 degrees
- moved JP1 29.3 mm to (-26.8, 20.3)
- moved C9 29.2 mm to (-23.7, 12.1), turned to 180 degrees
- moved U1 29.1 mm to (-21.8, 8.00)
- moved IC2 18.5 mm to (18.4, 9.65)
- moved BIPOUT+ 13.8 mm to (24.1, 41.7)
- moved BIPOUT- 13.8 mm to (24.1, 43.7)
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Connections:
- removed net +5V: C11.2, JP1.1, U2.1, U2.3
- removed net CS_CS: IC2.12, JP4.2
- removed net CS_IN: IC1.12, JP4.1
- new net +3V3: BOOT0.3, BOOT1.3, C11.2, C15.2, C16.2, C17.2, C20.2, C22.2, C23.2, JP1.1, SWD.4, U$1.1, U$1.13, U$1.19, U$1.32, U$1.48, U$1.64, U2.1, U2.3
- new net AQA: IC1.1, ICA.2, R12.1
- new net BOOT0: R51.2, U$1.60
- new net BOOT1: R52.2, U$1.28
- new net CS: U$1.54
- new net CSPOW: ICPOW.14
- new net DAC1: U$1.20
- new net LED1: PB12.A, U$1.33
- new net LED2: PB13.A, U$1.34
- new net LED3: PB14.A, U$1.35
- new net LED4: PB15.A, U$1.36
- new net N$13: C14.2, ICA.5
- new net N$15: IC1.2, R10.1, R11.1
- new net N$16: IC1.5, R13.1, R16.2
- new net N$18: IC1.9, R18.1, R19.1
- new net N$19: IC1.10, R17.1, R20.2
- new net N$21: IC1.3, R12.2, R9.1
- new net N$22: IC1.13, R22.1, R23.1
- new net N$23: IC1.12, R21.1, R24.2
- new net N$24: IC2.2, R26.1, R27.1
- new net N$25: IC2.3, R25.1, R28.2
- new net N$26: IC1.6, R14.1, R15.1
- new net N$27: IC2.6, R30.1, R31.1
- new net N$28: IC2.5, R29.1, R32.2
- new net N$29: IC2.9, R34.1, R35.1
- new net N$30: IC2.10, R33.1, R36.2
- new net N$31: IC2.13, R38.1, R39.1
- new net N$32: IC2.12, R37.1, R40.2
- new net N$33: C19.2, U$1.31
- new net N$34: IC1.7, R16.1
- new net N$35: IC1.8, R20.1
- new net N$36: IC1.14, R24.1
- new net N$37: C21.2, U$1.47
- new net N$38: IC2.7, R32.1
- new net N$39: IC2.8, R36.1
- new net N$40: IC2.14, R40.1
- new net N$41: R41.2, UTXL.C
- new net N$42: R42.2, URXL.C
- new net N$47: PB12.C, R47.2
- new net N$48: PB13.C, R48.2
- new net N$49: PB14.C, R49.2
- new net N$50: PB15.C, R50.2
- new net N$51: BOOT0.2, R51.1
- new net N$52: BOOT1.2, R52.1
- new net NRST: C29.2, SW1.2, SWD.1, U$1.7
- new net Q1: R9.2
- new net Q10: R26.2
- new net Q11: R29.2
- new net Q12: R30.2
- new net Q13: R33.2
- new net Q14: R34.2
- new net Q15: R37.2
- new net Q16: R38.2
- new net Q2: R10.2
- new net Q3: R13.2
- new net Q4: R14.2
- new net Q5: R17.2
- new net Q6: R18.2
- new net Q7: R21.2
- new net Q8: R22.2
- new net Q9: R25.2
- new net RCC1: C26.1, U$1.5, X1.1
- new net RCC2: C25.2, U$1.6, X1.3
- new net RTC1: C27.1, U$1.3, X2.2
- new net RTC2: C28.2, U$1.4, X2.1
- new net SWCLK: SWD.2, U$1.49
- new net SWDIO: SWD.3, U$1.46
- new net URX: U$1.43, URXL.A
- new net UTX: U$1.42, UTXL.A
- net +2V5: now also IC1.4, IC2.4, ICA.1; no longer IC1.10, IC1.16, IC2.10, IC2.16
- net -2V5: now also IC1.11, IC2.11, ICA.4
- net AQB: no longer IC1.1
- net AQC: no longer IC1.2
- net AQD: no longer IC1.3
- net AQE: now also IC2.1, R28.1; no longer IC1.4
- net AQF: no longer IC1.5
- net AQG: no longer IC1.6
- net AQH: no longer IC1.7
- net CSA: now also ICA.10; no longer IC2.15, ICPOW.14
- net CSB: no longer IC2.1
- net CSC: no longer IC2.2
- net CSD: no longer IC2.3
- net CSE: no longer IC2.4
- net CSF: no longer IC2.5
- net CSG: no longer IC2.6
- net CSH: no longer IC2.7
- net GND: now also BOOT0.1, BOOT1.1, BOOT2.1, C14.1, C15.1, C16.1, C17.1, C19.1, C20.1, C21.1, C22.1, C23.1, C25.1, C26.2, C27.2, C28.1, C29.1, ICA.6, R11.2, R15.2, R19.2, R23.2, R27.2, R31.2, R35.2, R39.2, R41.1, R42.1, R47.1, R48.1, R49.1, R50.1, SW1.1, SWD.5, SWD.6, U$1.12, U$1.18, U$1.63, X1.2, X1.4; no longer IC1.13, IC1.8, IC2.13, IC2.8, JP4.6
- net MISO: now also ICA.7, U$1.52; no longer JP4.3
- net MOSI: now also ICA.8, U$1.53; no longer IC1.14, IC2.14, JP4.4
- net SCLK: now also ICA.9, U$1.51; no longer IC1.11, IC2.11, JP4.5
- net W: now also ICA.3
Routing:
- net MOSI: track 112.0 -> 0.00 mm, vias 9 -> 0
- net +2V5: track 145.7 -> 37.2 mm, vias 12 -> 8
- net SCLK: track 105.8 -> 0.00 mm, vias 8 -> 0
- net -2V5: track 108.1 -> 46.9 mm, vias 13 -> 8
- net MISO: track 41.4 -> 0.00 mm, vias 7 -> 0
- net CS_CS: track 35.9 -> 0.00 mm
- net CS_IN: track 19.7 -> 0.00 mm, vias 1 -> 0
- net OUT_BIP: track 18.1 -> 0.00 mm
- net W: track 41.2 -> 56.4 mm
- net CSA: track 14.9 -> 0.00 mm, vias 1 -> 0
- net +5V: track 13.6 -> 0.00 mm
- net LVLW: track 12.6 -> 0.00 mm, vias 1 -> 0
- net AQB: track 11.9 -> 0.00 mm, vias 1 -> 0
- net CSB: track 11.7 -> 0.00 mm
- net AQH: track 11.7 -> 0.00 mm, vias 1 -> 0
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Other:
- board size 40.6 x 48.3 mm -> 50.8 x 50.8 mm

Commit message: Almost finished neuron v2
Parts:
- removed BOOT2: (no value), pinhead:1X03
- removed JP2: (no value), pinhead:1X01
- added UART1: (no value), pinhead:1X03
- moved C25 256.9 mm to (41.3, 22.7), turned to 90 degrees
- moved C28 252.0 mm to (36.4, 23.6), flipped to the bottom, turned to 180 degrees
- moved C29 251.1 mm to (36.8, 14.0), turned to 180 degrees
- moved C26 250.9 mm to (38.1, 17.4)
- moved C27 246.8 mm to (36.3, 17.9), flipped to the bottom
- moved X2 228.4 mm to (37.5, 20.8), flipped to the bottom, turned to 270 degrees
- moved SW1 221.5 mm to (36.8, 11.4), turned to 180 degrees
- moved SWD 209.6 mm to (22.9, 12.7)
- moved X1 200.0 mm to (38.4, 21.6), turned to 90 degrees
- moved C21 189.9 mm to (-17.8, -43.2)
- moved R40 165.2 mm to (10.8, 45.0)
- moved R39 162.3 mm to (13.8, 40.9)
- moved R37 161.3 mm to (13.8, 45.0)
- moved R38 158.5 mm to (13.8, 42.9)
- moved R35 140.5 mm to (13.8, 37.8)
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Connections:
- removed net CS: U$1.54
- removed net DAC1: U$1.20
- removed net N$31: IC2.13, R38.1, R39.1
- removed net N$34: IC1.7, R16.1
- removed net N$35: IC1.8, R20.1
- removed net N$36: IC1.14, R24.1
- removed net N$38: IC2.7, R32.1
- removed net N$39: IC2.8, R36.1
- removed net N$40: IC2.14, R40.1
- new net N$43: IC2.2, R25.1, R28.2
- new net N$45: U$1.58
- new net N$46: U$1.59
- new net N$53: U$1.61
- new net N$54: U$1.62
- net +2V5: now also BOOT0.3, BOOT1.3, C15.2, C16.2, C17.2, C20.2, C22.2, C23.2, SWD.4, U$1.1, U$1.13, U$1.19, U$1.32, U$1.48, U$1.64
- net +3V3: no longer BOOT0.3, BOOT1.3, C15.2, C16.2, C17.2, C20.2, C22.2, C23.2, SWD.4, U$1.1, U$1.13, U$1.19, U$1.32, U$1.48, U$1.64
- net AQB: now also IC1.14, R24.1
- net AQC: now also IC1.8, R20.1
- net AQD: now also IC1.7, R16.1
- net AQF: now also IC2.14, R40.1
- net AQG: now also IC2.8, R36.1
- net AQH: now also IC2.7, R32.1
- net GND: now also IC4.5, IC4.6, UART1.1; no longer BOOT2.1
- net MISO: now also U$1.22; no longer U$1.52
- net MOSI: now also U$1.23; no longer U$1.53
- net N$15: now also IC1.3; no longer IC1.2
- net N$16: now also IC1.6; no longer IC1.5
- net N$18: now also IC1.10; no longer IC1.9
- net N$19: now also IC1.9; no longer IC1.10
- net N$21: now also IC1.2; no longer IC1.3
- net N$22: now also IC1.12; no longer IC1.13
- net N$23: now also IC1.13; no longer IC1.12
- net N$24: now also IC2.3; no longer IC2.2
- net N$25: now also IC2.12, R38.1, R39.1; no longer IC2.3, R25.1, R28.2
- net N$26: now also IC1.5; no longer IC1.6
- net N$27: now also IC2.5; no longer IC2.6
- net N$28: now also IC2.6; no longer IC2.5
- net N$29: now also IC2.10; no longer IC2.9
- net N$30: now also IC2.9; no longer IC2.10
- net N$32: now also IC2.13; no longer IC2.12
- net OUT: now also U$1.11; no longer JP2.1
- net Q1: now also U$1.57
- net Q10: now also U$1.52
- net Q11: now also U$1.50
- net Q12: now also U$1.51
- net Q2: now also U$1.56
- net Q3: now also U$1.54
- net Q4: now also U$1.55
- net Q9: now also U$1.53
- net SCLK: now also U$1.21; no longer U$1.51
- net URX: now also UART1.2
- net UTX: now also UART1.3
Routing:
- net +2V5: track 37.2 -> 226.3 mm, vias 8 -> 17
- net -2V5: track 46.9 -> 192.6 mm, vias 8 -> 15
- net MISO: track 0.00 -> 71.8 mm, vias 0 -> 9
- net MOSI: track 0.00 -> 67.1 mm, vias 0 -> 10
- net SCLK: track 0.00 -> 57.4 mm, vias 0 -> 9
- net OUT: track 0.00 -> 41.4 mm
- net AQH: track 0.00 -> 23.9 mm
- net AQA: track 0.00 -> 23.7 mm
- net AQG: track 0.00 -> 23.0 mm
- net AQB: track 0.00 -> 22.9 mm
- net AQD: track 0.00 -> 22.7 mm
- net AQE: track 0.00 -> 22.7 mm
- net AQC: track 0.00 -> 22.0 mm
- net AQF: track 0.00 -> 20.8 mm
- net NRST: track 0.00 -> 18.5 mm
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Other:
- board size 50.8 x 50.8 mm -> 50.8 x 71.1 mm

Commit message: finished v1
Parts:
- removed JP1, UART1: (no value), pinhead:1X03
- removed PB12, PB13, PB14, PB15, URXL, UTXL: LEDCHIPLED_0805, audio amplifier example:CHIPLED_0805
- removed SWD: B6B-ZR, jst:B6B-ZR
- added C18, C24: 2.2 u, rcl:C0603K
- added IC5: 74HC595D, 74xx-eu:SO16
- added JP10, JP11, JP9: (no value), pinhead:1X06
- added P30, P31, P46, P47, SWDIO: JUMPER-SMT_3_2-NC_PASTE_NO-SILK, SparkFun-Jumpers:SMT-JUMPER_3_2-NC_PASTE_NO-SILK
- added PC0, PC1, PC2, PC3, URXL1, URXL2, UTXL1, UTXL2: LEDCHIPLED_0805, audio amplifier example:CHIPLED_0805
- added R43, R44: 180R, rcl:R0603
- BOOT0, BOOT1: value (none) -> JUMPER-SMT_3_2-NC_PASTE_NO-SILK; device pinhead:1X03 -> SparkFun-Jumpers:SMT-JUMPER_3_2-NC_PASTE_NO-SILK
- moved R47 268.1 mm to (59.3, 38.0), turned to 270 degrees
- moved R48 266.0 mm to (56.5, 38.0), turned to 270 degrees
- moved R49 264.3 mm to (53.8, 38.0), turned to 270 degrees
- moved R50 262.9 mm to (51.1, 38.0), turned to 270 degrees
- moved C23 261.1 mm to (44.1, 33.8), turned to 180 degrees
- moved C16 260.5 mm to (33.0, 33.0), turned to 270 degrees
- moved C22 259.3 mm to (51.1, 31.8), turned to 180 degrees
- moved BOOT1 256.0 mm to (46.6, 36.2)
- moved C19 255.1 mm to (18.2, 21.5), turned to 90 degrees
- moved R52 254.4 mm to (45.8, 32.1), turned to 180 degrees
- moved C20 247.4 mm to (45.1, 19.8), turned to 90 degrees
- moved C17 247.1 mm to (30.0, 19.8), turned to 90 degrees
- moved R41 246.6 mm to (10.5, 30.5), turned to 270 degrees
- moved C15 245.8 mm to (41.9, 17.4), turned to 90 degrees
- moved R51 240.0 mm to (38.4, 17.8)
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Connections:
- removed net LED1: PB12.A, U$1.33
- removed net LED2: PB13.A, U$1.34
- removed net LED3: PB14.A, U$1.35
- removed net LED4: PB15.A, U$1.36
- removed net N$33: C19.2, U$1.31
- removed net N$37: C21.2, U$1.47
- removed net URX: U$1.43, UART1.2, URXL.A
- removed net UTX: U$1.42, UART1.3, UTXL.A
- new net CS_CS: IC5.12, U$1.20
- new net N$34: R43.2, UTXL2.C
- new net N$35: R44.2, URXL2.C
- new net N$36: C21.2, P47.3
- new net N$38: C18.2, P31.3
- new net N$51: C19.2, P46.3
- new net N$55: C24.2, P30.3
- new net N$56: PC3.A, U$1.11
- new net N$57: PC2.A, U$1.10
- new net N$58: PC1.A, U$1.9
- new net N$59: PC0.A, U$1.8
- new net P30: P30.2, U$1.30
- new net P31: P31.2, U$1.31
- new net P45: SWDIO.1, U$1.45
- new net P46: P46.2, SWDIO.3, U$1.46
- new net P47: P47.2, U$1.47
- new net URX1: JP10.4, U$1.43, URXL1.A
- new net URX2: JP9.5, U$1.17, URXL2.A
- new net UTX1: JP10.5, U$1.42, UTXL1.A
- new net UTX2: JP9.4, U$1.16, UTXL2.A
- net +2V5: now also BOOT0.1, BOOT1.1, IC5.10, IC5.16, JP11.4; no longer BOOT0.3, BOOT1.3, SWD.4
- net +3V3: now also JP10.1, JP9.1; no longer JP1.1
- net -5V: now also JP10.3, JP9.3; no longer JP1.3
- net CSA: now also IC5.15
- net CSB: now also IC5.1
- net CSC: now also IC5.2
- net CSD: now also IC5.3
- net CSE: now also IC5.4
- net CSF: now also IC5.5
- net CSG: now also IC5.6
- net CSH: now also IC5.7
- net GND: now also BOOT0.3, BOOT1.3, C18.1, C24.1, IC5.13, IC5.8, JP10.2, JP10.6, JP11.5, JP11.6, JP9.2, JP9.6, P30.1, P31.1, P46.1, P47.1, R43.1, R44.1; no longer BOOT0.1, BOOT1.1, JP1.2, SWD.5, SWD.6, UART1.1
- net MOSI: now also IC5.14
- net N$41: now also URXL1.C; no longer UTXL.C
- net N$42: now also UTXL1.C; no longer URXL.C
- net N$47: now also PC0.C; no longer PB12.C
- net N$48: now also PC1.C; no longer PB13.C
- net N$49: now also PC2.C; no longer PB14.C
- net N$50: now also PC3.C; no longer PB15.C
- net NRST: now also JP11.1; no longer SWD.1
- net OUT: now also U$1.15; no longer U$1.11
- net Q1: now also U$1.50; no longer U$1.57
- net Q10: now also U$1.38; no longer U$1.52
- net Q11: now also U$1.36; no longer U$1.50
- net Q12: now also U$1.37; no longer U$1.51
- net Q13: now also U$1.35
- net Q14: now also U$1.34
- net Q15: now also U$1.29
- net Q16: now also U$1.33
- net Q2: now also U$1.44; no longer U$1.56
- net Q3: now also U$1.40; no longer U$1.54
- net Q4: now also U$1.41; no longer U$1.55
- net Q5: now also U$1.27
- net Q6: now also U$1.26
- net Q7: now also U$1.24
- net Q8: now also U$1.25
- net Q9: now also U$1.39; no longer U$1.53
- net RTC1: now also U$1.4; no longer U$1.3
- net RTC2: now also U$1.3; no longer U$1.4
- net SCLK: now also IC5.11
- net SWCLK: now also JP11.2; no longer SWD.2
- net SWDIO: now also JP11.3, SWDIO.2; no longer SWD.3, U$1.46
Routing:
- net +3V3: track 12.0 -> 125.9 mm
- net +2V5: track 226.3 -> 329.3 mm, vias 17 -> 20
- net -5V: track 11.1 -> 109.0 mm, vias 0 -> 2
- net Q1: track 0.00 -> 65.2 mm, vias 0 -> 2
- net Q2: track 0.00 -> 57.3 mm
- net Q4: track 0.00 -> 48.4 mm
- net OUT: track 41.4 -> 86.4 mm
- net Q3: track 0.00 -> 44.8 mm
- net Q7: track 0.00 -> 42.7 mm, vias 0 -> 2
- net Q8: track 0.00 -> 40.0 mm, vias 0 -> 2
- net Q9: track 0.00 -> 38.7 mm
- net Q10: track 0.00 -> 35.9 mm
- net Q6: track 0.00 -> 34.2 mm, vias 0 -> 2
- net Q5: track 0.00 -> 31.4 mm, vias 0 -> 2
- net UTX1: track 0.00 -> 31.2 mm, vias 0 -> 2
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Other:
- board size 50.8 x 71.1 mm -> 67.3 x 87.6 mm

Commit message: some patches
Parts:
- BOOT0, BOOT1, P30, P31, P46, P47, SWDIO: value JUMPER-SMT_3_2-NC_PASTE_NO-SILK -> JUMPER-SMT_3_NO_NO-SILK; device SparkFun-Jumpers:SMT-JUMPER_3_2-NC_PASTE_NO-SILK -> SparkFun-Jumpers_custom:SMT-JUMPER_3_NO_NO-SILK
- moved R4 5.98 mm to (12.2, 17.4), turned to 0 degrees
- moved R52 5.59 mm to (40.3, 32.0)
- moved C21 5.38 mm to (18.9, 18.4), turned to 90 degrees
- moved C19 5.33 mm to (12.8, 21.5)
- moved P30 5.21 mm to (21.3, 30.5)
- moved BOOT0 5.08 mm to (32.4, 15.4)
- moved C22 5.08 mm to (46.0, 31.8)
- moved C23 5.08 mm to (39.0, 33.8)
- moved C25 5.08 mm to (43.1, 26.4)
- moved C26 5.08 mm to (51.2, 26.7)
- moved PC3 5.08 mm to (46.0, 34.3)
- moved R50 5.08 mm to (46.0, 38.0)
- moved URXL2 5.08 mm to (54.1, 21.6)
- moved UTXL2 5.08 mm to (54.1, 25.4)
- moved C11 5.08 mm to (25.4, 6.48)
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Connections:
- removed net N$45: U$1.58
- removed net N$46: U$1.59
- removed net N$53: U$1.61
- removed net N$54: U$1.62
- net CSPOW: now also U$1.15
- net OUT: now also U$1.14; no longer U$1.15
Routing:
- net CSPOW: track 0.00 -> 57.6 mm, vias 0 -> 2
- net +2V5: track 329.3 -> 336.1 mm
- net +3V3: track 125.9 -> 120.2 mm, vias 0 -> 2
- net N$52: track 0.00 -> 4.36 mm
- net -5V: track 109.0 -> 105.1 mm, vias 2 -> 4
- net URX1: track 28.3 -> 25.2 mm
- net UTX1: track 31.2 -> 28.4 mm
- net N$34: track 0.00 -> 2.54 mm
- net OUT: track 86.4 -> 87.5 mm
- net -2V5: track 164.1 -> 163.0 mm
- net URX2: track 25.3 -> 26.4 mm
- net NRST: track 28.6 -> 29.5 mm
- net W: track 70.4 -> 71.1 mm
- net P45: track 4.80 -> 5.46 mm
Other:
- board size 67.3 x 87.6 mm -> 61 x 87.6 mm
- board text added: "+3"
- board text added: "-3"
- board text added: "P45"
- board text added: "P46"
