File: neuron.sch (EAGLE design)
At the start: 112 parts, among them IC1 AD8684RU, IC2 AD8684RU, IC3 ADA4692-2R, IC4 ADA4692-2R, SW1 B3U-1000P, U1 TPS72301DBVRSOT-23-5, U2 TLV703, X1 ABM3B-16.000MHZ-B2-T, X2 9HT10-32.768KDZF-T

Commit message: Almost finished neuron v2
Parts:
- removed JP2: (no value), pinhead:PINHD-1X1
- renumbered BOOT2 to UART1
Connections:
- removed net CS: U$1.PD2/SDIO_CMD
- removed net DAC1: U$1.PA4/SPI1_NSS
- removed net N$31: IC2D.-IN, R38.1, R39.1
- removed net N$34: IC1B.OUT, R16.1
- removed net N$35: IC1C.OUT, R20.1
- removed net N$36: IC1D.OUT, R24.1
- removed net N$38: IC2B.OUT, R32.1
- removed net N$39: IC2C.OUT, R36.1
- removed net N$40: IC2D.OUT, R40.1
- new net N$43: IC2A.-IN, R25.1, R28.2
- new net N$45: U$1.PB6
- new net N$46: U$1.PB7
- new net N$53: U$1.PB8
- new net N$54: U$1.PB9
- net +2V5: now also BOOT0.3, BOOT1.3, C15.2, C16.2, C17.2, C20.2, C22.2, C23.2, SWD.4, U$1.VBAT, U$1.VDD1, U$1.VDD2, U$1.VDD3, U$1.VDD4, U$1.VDDA
- net +3V3: no longer BOOT0.3, BOOT1.3, C15.2, C16.2, C17.2, C20.2, C22.2, C23.2, SWD.4, U$1.VBAT, U$1.VDD1, U$1.VDD2, U$1.VDD3, U$1.VDD4, U$1.VDDA
- net AQB: now also IC1D.OUT, R24.1
- net AQC: now also IC1C.OUT, R20.1
- net AQD: now also IC1B.OUT, R16.1
- net AQF: now also IC2D.OUT, R40.1
- net AQG: now also IC2C.OUT, R36.1
- net AQH: now also IC2B.OUT, R32.1
- net GND: now also IC4B.IN+, IC4B.IN-
- net MISO: now also U$1.PA6/SPI1_MISO; no longer U$1.PC11/SDIO_D3
- net MOSI: now also U$1.PA7/SPI1_MOSI; no longer U$1.PC12/SDIO_CLK
- net N$15: now also IC1A.+IN; no longer IC1A.-IN
- net N$16: now also IC1B.-IN; no longer IC1B.+IN
- net N$18: now also IC1C.+IN; no longer IC1C.-IN
- net N$19: now also IC1C.-IN; no longer IC1C.+IN
- net N$21: now also IC1A.-IN; no longer IC1A.+IN
- net N$22: now also IC1D.+IN; no longer IC1D.-IN
- net N$23: now also IC1D.-IN; no longer IC1D.+IN
- net N$24: now also IC2A.+IN; no longer IC2A.-IN
- net N$25: now also IC2D.+IN, R38.1, R39.1; no longer IC2A.+IN, R25.1, R28.2
- net N$26: now also IC1B.+IN; no longer IC1B.-IN
- net N$27: now also IC2B.+IN; no longer IC2B.-IN
- net N$28: now also IC2B.-IN; no longer IC2B.+IN
- net N$29: now also IC2C.+IN; no longer IC2C.-IN
- net N$30: now also IC2C.-IN; no longer IC2C.+IN
- net N$32: now also IC2D.-IN; no longer IC2D.+IN
- net OUT: now also U$1.PC3; no longer JP2.1
- net Q1: now also U$1.PB5
- net Q10: now also U$1.PC11/SDIO_D3
- net Q11: now also U$1.PA15/JTDI
- net Q12: now also U$1.PC10/SDIO_D2
- net Q2: now also U$1.PB4/JTRST
- net Q3: now also U$1.PD2/SDIO_CMD
- net Q4: now also U$1.PB3/JTDO
- net Q9: now also U$1.PC12/SDIO_CLK
- net SCLK: now also U$1.PA5/SPI1_SCK; no longer U$1.PC10/SDIO_D2
- net URX: now also UART1.2
- net UTX: now also UART1.3
Other:
- moved on the sheet: IC1A, IC1B, IC1C, IC1D, IC2A, IC2B, IC2C, IC2D

Commit message: finished v1
Parts:
- removed JP1, UART1: (no value), pinhead:PINHD-1X3
- removed PB12, PB13, PB14, PB15: LEDCHIPLED_0805, audio amplifier example:LEDCHIPLED_0805
- removed SWD: B6B-ZR, jst:B6B-ZR
- added C18, C24: 2.2 u, rcl:C-EUC0603K
- added IC5: 74HC595D, 74xx-eu:74HC595D
- added JP10, JP11, JP9: (no value), pinhead:PINHD-1X6
- added P30, P31, P46, P47, SWDIO: JUMPER-SMT_3_2-NC_PASTE_NO-SILK, SparkFun-Jumpers:JUMPER-SMT_3_2-NC_PASTE_NO-SILK
- added PC0, PC1, PC2, PC3, URXL2, UTXL2: LEDCHIPLED_0805, audio amplifier example:LEDCHIPLED_0805
- added R43, R44: 180R, rcl:R-EU_R0603
- BOOT0, BOOT1: value (none) -> JUMPER-SMT_3_2-NC_PASTE_NO-SILK; device pinhead:PINHD-1X3 -> SparkFun-Jumpers:JUMPER-SMT_3_2-NC_PASTE_NO-SILK
- renumbered URXL to UTXL1, UTXL to URXL1
Connections:
- removed net LED1: PB12.A, U$1.PB12/I2S2_WS
- removed net LED2: PB13.A, U$1.PB13/I2S2_CK
- removed net LED3: PB14.A, U$1.PB14/I2S2_XD
- removed net LED4: PB15.A, U$1.PB15/I2S2_SD
- removed net N$33: C19.2, U$1.VCAP1
- removed net N$37: C21.2, U$1.VCAP2
- removed net URX: U$1.PA10/UART1_RX, UART1.2, UTXL1.A
- removed net UTX: U$1.PA9/UART1_TX, UART1.3, URXL1.A
- new net CS_CS: IC5A.RCK, U$1.PA4/SPI1_NSS
- new net N$34: R43.2, UTXL2.C
- new net N$35: R44.2, URXL2.C
- new net N$36: C21.2, P47.3
- new net N$38: C18.2, P31.3
- new net N$51: C19.2, P46.3
- new net N$55: C24.2, P30.3
- new net N$56: PC3.A, U$1.PC3
- new net N$57: PC2.A, U$1.PC2
- new net N$58: PC1.A, U$1.PC1
- new net N$59: PC0.A, U$1.PC0
- new net P30: P30.2, U$1.PB11
- new net P31: P31.2, U$1.VCAP1
- new net P45: SWDIO.1, U$1.PA12
- new net P46: P46.2, SWDIO.3, U$1.PA13/JTMS
- new net P47: P47.2, U$1.VCAP2
- new net URX1: JP10.4, U$1.PA10/UART1_RX, URXL1.A
- new net URX2: JP9.5, U$1.PA3/UART2_RX, URXL2.A
- new net UTX1: JP10.5, U$1.PA9/UART1_TX, UTXL1.A
- new net UTX2: JP9.4, U$1.PA2/UART2_TX, UTXL2.A
- net +2V5: now also BOOT0.1, BOOT1.1, IC5A.SCL, IC5P.VCC, JP11.4; no longer BOOT0.3, BOOT1.3, SWD.4
- net +3V3: now also JP10.1, JP9.1; no longer JP1.1
- net -5V: now also JP10.3, JP9.3; no longer JP1.3
- net CSA: now also IC5A.QA
- net CSB: now also IC5A.QB
- net CSC: now also IC5A.QC
- net CSD: now also IC5A.QD
- net CSE: now also IC5A.QE
- net CSF: now also IC5A.QF
- net CSG: now also IC5A.QG
- net CSH: now also IC5A.QH
- net GND: now also BOOT0.3, BOOT1.3, C18.1, C24.1, IC5A.G, IC5P.GND, JP10.2, JP10.6, JP11.5, JP11.6, JP9.2, JP9.6, P30.1, P31.1, P46.1, P47.1, R43.1, R44.1; no longer BOOT0.1, BOOT1.1, JP1.2, SWD.5, SWD.6, UART1.1
- net MOSI: now also IC5A.SER
- net N$47: now also PC0.C; no longer PB12.C
- net N$48: now also PC1.C; no longer PB13.C
- net N$49: now also PC2.C; no longer PB14.C
- net N$50: now also PC3.C; no longer PB15.C
- net NRST: now also JP11.1; no longer SWD.1
- net OUT: now also U$1.PA1; no longer U$1.PC3
- net Q1: now also U$1.PA15/JTDI; no longer U$1.PB5
- net Q10: now also U$1.PC7; no longer U$1.PC11/SDIO_D3
- net Q11: now also U$1.PB15/I2S2_SD; no longer U$1.PA15/JTDI
- net Q12: now also U$1.PC6/I2S2_MCK; no longer U$1.PC10/SDIO_D2
- net Q13: now also U$1.PB14/I2S2_XD
- net Q14: now also U$1.PB13/I2S2_CK
- net Q15: now also U$1.PB10
- net Q16: now also U$1.PB12/I2S2_WS
- net Q2: now also U$1.PA11; no longer U$1.PB4/JTRST
- net Q3: now also U$1.PC9/SDIO_D1; no longer U$1.PD2/SDIO_CMD
- net Q4: now also U$1.PA8; no longer U$1.PB3/JTDO
- net Q5: now also U$1.PB1
- net Q6: now also U$1.PB0
- net Q7: now also U$1.PC4
- net Q8: now also U$1.PC5
- net Q9: now also U$1.PC8/SDIO_D0; no longer U$1.PC12/SDIO_CLK
- net RTC1: now also U$1.PC15; no longer U$1.PC14
- net RTC2: now also U$1.PC14; no longer U$1.PC15
- net SCLK: now also IC5A.SCK
- net SWCLK: now also JP11.2; no longer SWD.2
- net SWDIO: now also JP11.3, SWDIO.2; no longer SWD.3, U$1.PA13/JTMS
Other:
- moved on the sheet: C19, C21, C23, R47, R48, R49, R50

Commit message: some patches
Parts:
- BOOT0, BOOT1, P30, P31, P46, P47, SWDIO: value JUMPER-SMT_3_2-NC_PASTE_NO-SILK -> JUMPER-SMT_3_NO_NO-SILK; device SparkFun-Jumpers:JUMPER-SMT_3_2-NC_PASTE_NO-SILK -> SparkFun-Jumpers_custom:JUMPER-SMT_3_NO_NO-SILK
Connections:
- removed net N$45: U$1.PB6
- removed net N$46: U$1.PB7
- removed net N$53: U$1.PB8
- removed net N$54: U$1.PB9
- net CSPOW: now also U$1.PA1
- net OUT: now also U$1.PA0; no longer U$1.PA1
Changed lines of the file:
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@@
 <part name="IC1" library="linear" library_urn="urn:adsk.eagle:library:262" deviceset="AD8684" device="RU" package3d_urn="urn:adsk.eagle:package:16437/2"/>
 <part name="IC2" library="linear" library_urn="urn:adsk.eagle:library:262" deviceset="AD8684" device="RU" package3d_urn="urn:adsk.eagle:package:16437/2"/>
-<part name="U$1" library="SparkFun-IC-Microcontroller" deviceset="STM32F405RG" device="" override_package3d_urn="urn:adsk.eagle:package:17075202/2" override_package_urn="urn:adsk.eagle:footprint:17075203/1" value="STM32F405RGT6"/>
+<part name="U$1" library="SparkFun-IC-Microcontroller" library_urn="urn:adsk.eagle:library:525" deviceset="STM32F405RG" device="" package3d_urn="urn:adsk.eagle:package:38936/1" override_package3d_urn="urn:adsk.eagle:package:17075202/2" override_package_urn="urn:adsk.eagle:footprint:17075203/1" override_locally_modified="yes" value="STM32F405RGT6"/>
 <part name="C15" library="rcl" library_urn="urn:adsk.eagle:library:334" deviceset="C-EU" device="C0603K" package3d_urn="urn:adsk.eagle:package:23680/2" value="100n"/>
 <part name="C16" library="rcl" library_urn="urn:adsk.eagle:library:334" deviceset="C-EU" device="C0603K" package3d_urn="urn:adsk.eagle:package:23680/2" value="100n"/>
@@
 <part name="+3V22" library="untitled" deviceset="+2V5" device=""/>
 <part name="+3V23" library="untitled" deviceset="+2V5" device=""/>
-<part name="BOOT0" library="SparkFun-Jumpers" library_urn="urn:adsk.eagle:library:528" deviceset="JUMPER-SMT_3_2-NC_PASTE" device="_NO-SILK" package3d_urn="urn:adsk.eagle:package:39292/1"/>
-<part name="BOOT1" library="SparkFun-Jumpers" library_urn="urn:adsk.eagle:library:528" deviceset="JUMPER-SMT_3_2-NC_PASTE" device="_NO-SILK" package3d_urn="urn:adsk.eagle:package:39292/1"/>
+<part name="BOOT0" library="SparkFun-Jumpers_custom" deviceset="JUMPER-SMT_3_NO" device="_NO-SILK" package3d_urn="urn:adsk.eagle:package:39284/1"/>
+<part name="BOOT1" library="SparkFun-Jumpers_custom" deviceset="JUMPER-SMT_3_NO" device="_NO-SILK" package3d_urn="urn:adsk.eagle:package:39284/1"/>
 <part name="GND50" library="supply1" library_urn="urn:adsk.eagle:library:371" deviceset="GND" device=""/>
 <part name="UTXL2" library="audio amplifier example" library_urn="urn:adsk.eagle:library:970892" deviceset="LED" device="CHIPLED_0805" package3d_urn="urn:adsk.eagle:package:970933/2"/>
@@
 <part name="R44" library="rcl" library_urn="urn:adsk.eagle:library:334" deviceset="R-EU_" device="R0603" package3d_urn="urn:adsk.eagle:package:23555/3" value="180R"/>
 <part name="GND55" library="supply1" library_urn="urn:adsk.eagle:library:371" deviceset="GND" device=""/>
-<part name="P47" library="SparkFun-Jumpers" library_urn="urn:adsk.eagle:library:528" deviceset="JUMPER-SMT_3_2-NC_PASTE" device="_NO-SILK" package3d_urn="urn:adsk.eagle:package:39292/1"/>
+<part name="P47" library="SparkFun-Jumpers_custom" deviceset="JUMPER-SMT_3_NO" device="_NO-SILK" package3d_urn="urn:adsk.eagle:package:39284/1"/>
 <part name="GND56" library="supply1" library_urn="urn:adsk.eagle:library:371" deviceset="GND" device=""/>
 <part name="C18" library="rcl" library_urn="urn:adsk.eagle:library:334" deviceset="C-EU" device="C0603K" package3d_urn="urn:adsk.eagle:package:23680/2" value="2.2 u"/>
 <part name="GND34" library="supply1" library_urn="urn:adsk.eagle:library:371" deviceset="GND" device=""/>
-<part name="P31" library="SparkFun-Jumpers" library_urn="urn:adsk.eagle:library:528" deviceset="JUMPER-SMT_3_2-NC_PASTE" device="_NO-SILK" package3d_urn="urn:adsk.eagle:package:39292/1"/>
+<part name="P31" library="SparkFun-Jumpers_custom" deviceset="JUMPER-SMT_3_NO" device="_NO-SILK" package3d_urn="urn:adsk.eagle:package:39284/1"/>
 <part name="GND58" library="supply1" library_urn="urn:adsk.eagle:library:371" deviceset="GND" device=""/>
-<part name="SWDIO" library="SparkFun-Jumpers" library_urn="urn:adsk.eagle:library:528" deviceset="JUMPER-SMT_3_2-NC_PASTE" device="_NO-SILK" package3d_urn="urn:adsk.eagle:package:39292/1"/>
+<part name="SWDIO" library="SparkFun-Jumpers_custom" deviceset="JUMPER-SMT_3_NO" device="_NO-SILK" package3d_urn="urn:adsk.eagle:package:39284/1"/>
 <part name="C19" library="rcl" library_urn="urn:adsk.eagle:library:334" deviceset="C-EU" device="C0603K" package3d_urn="urn:adsk.eagle:package:23680/2" value="2.2 u"/>
 <part name="GND59" library="supply1" library_urn="urn:adsk.eagle:library:371" deviceset="GND" device=""/>
-<part name="P46" library="SparkFun-Jumpers" library_urn="urn:adsk.eagle:library:528" deviceset="JUMPER-SMT_3_2-NC_PASTE" device="_NO-SILK" package3d_urn="urn:adsk.eagle:package:39292/1"/>
+<part name="P46" library="SparkFun-Jumpers_custom" deviceset="JUMPER-SMT_3_NO" device="_NO-SILK" package3d_urn="urn:adsk.eagle:package:39284/1"/>
 <part name="GND60" library="supply1" library_urn="urn:adsk.eagle:library:371" deviceset="GND" device=""/>
 <part name="C24" library="rcl" library_urn="urn:adsk.eagle:library:334" deviceset="C-EU" device="C0603K" package3d_urn="urn:adsk.eagle:package:23680/2" value="2.2 u"/>
 <part name="GND61" library="supply1" library_urn="urn:adsk.eagle:library:371" deviceset="GND" device=""/>
-<part name="P30" library="SparkFun-Jumpers" library_urn="urn:adsk.eagle:library:528" deviceset="JUMPER-SMT_3_2-NC_PASTE" device="_NO-SILK" package3d_urn="urn:adsk.eagle:package:39292/1"/>
+<part name="P30" library="SparkFun-Jumpers_custom" deviceset="JUMPER-SMT_3_NO" device="_NO-SILK" package3d_urn="urn:adsk.eagle:package:39284/1"/>
 <part name="GND62" library="supply1" library_urn="urn:adsk.eagle:library:371" deviceset="GND" device=""/>
 <part name="JP9" library="pinhead" library_urn="urn:adsk.eagle:library:325" deviceset="PINHD-1X6" device="" package3d_urn="urn:adsk.eagle:package:22472/2"/>
 <part name="JP10" library="pinhead" library_urn="urn:adsk.eagle:library:325" deviceset="PINHD-1X6" device="" package3d_urn="urn:adsk.eagle:package:22472/2"/>
 <part name="JP11" library="pinhead" library_urn="urn:adsk.eagle:library:325" deviceset="PINHD-1X6" device="" package3d_urn="urn:adsk.eagle:package:22472/2"/>
-<part name="IC5" library="74xx-eu" library_urn="urn:adsk.eagle:library:85" deviceset="74*595" device="D" package3d_urn="urn:adsk.eagle:package:2010/1" technology="HC"/>
+<part name="IC5" library="74xx-eu" library_urn="urn:adsk.eagle:library:85" deviceset="74*595" device="D" package3d_urn="urn:adsk.eagle:package:2010/1" override_package3d_urn="urn:adsk.eagle:package:26760955/2" override_package_urn="urn:adsk.eagle:footprint:1637/1" technology="HC"/>
 <part name="GND20" library="supply1" library_urn="urn:adsk.eagle:library:371" deviceset="GND" device=""/>
 <part name="+3V20" library="untitled" deviceset="+2V5" device=""/>
@@
 <wire x1="60.96" y1="60.96" x2="60.96" y2="68.58" width="0.1524" layer="91"/>
 <wire x1="60.96" y1="68.58" x2="81.28" y2="68.58" width="0.1524" layer="91"/>
+<junction x="99.06" y="68.58"/>
 </segment>
 <segment>
@@
 </segment>
 <segment>
-<pinref part="U$1" gate="G$1" pin="PA1"/>
-<wire x1="139.7" y1="398.78" x2="132.08" y2="398.78" width="0.1524" layer="91"/>
-<label x="132.08" y="398.78" size="1.778" layer="95"/>
+<pinref part="U$1" gate="G$1" pin="PA0"/>
+<wire x1="139.7" y1="401.32" x2="132.08" y2="401.32" width="0.1524" layer="91"/>
+<label x="132.08" y="401.32" size="1.778" layer="95"/>
 </segment>
 </net>
@@
 <wire x1="149.86" y1="236.22" x2="160.02" y2="236.22" width="0.1524" layer="91"/>
 <label x="152.4" y="236.22" size="1.778" layer="95"/>
+</segment>
+<segment>
+<pinref part="U$1" gate="G$1" pin="PA1"/>
+<wire x1="139.7" y1="398.78" x2="132.08" y2="398.78" width="0.1524" layer="91"/>
+<label x="130.302" y="398.78" size="1.778" layer="95"/>
 </segment>
 </net>
@@
 </segment>
 </net>
-<net name="N$46" class="0">
-<segment>
-<pinref part="U$1" gate="G$1" pin="PB7"/>
-<wire x1="198.12" y1="421.64" x2="208.28" y2="421.64" width="0.1524" layer="91"/>
-</segment>
-</net>
-<net name="N$45" class="0">
-<segment>
-<pinref part="U$1" gate="G$1" pin="PB6"/>
-<wire x1="198.12" y1="419.1" x2="208.28" y2="419.1" width="0.1524" layer="91"/>
-</segment>
-</net>
-<net name="N$53" class="0">
-<segment>
-<pinref part="U$1" gate="G$1" pin="PB8"/>
-<wire x1="198.12" y1="426.72" x2="208.28" y2="426.72" width="0.1524" layer="91"/>
-</segment>
-</net>
-<net name="N$54" class="0">
-<segment>
-<pinref part="U$1" gate="G$1" pin="PB9"/>
-<wire x1="198.12" y1="429.26" x2="208.28" y2="429.26" width="0.1524" layer="91"/>
-</segment>
-</net>

Commit message: added firmware
Parts:
- removed IC1, IC2: AD8684RU, linear:AD8684RU
- added IC6, IC7: AD8609RU, analog-devices:AD8609RU
- C13: device rcl:C-EUC0805K -> rcl:C-EUC0603K
- C25, C26: value 18p -> 33p
- C27, C28: value 12.5p -> 22p
- R1, R2, R3: device rcl:R-EU_R0805 -> rcl:R-EU_R0603
- R4, R5, R6, R7, R8: value 200 -> 180R
Connections:
- removed net N$27: IC2B.+IN, R30.1, R31.1
- new net N$33: IC7B.IN+, R30.1, R31.1
- net +2V5: now also IC6P.V+, IC7P.V+; no longer IC1P.V+, IC2P.V+
- net -2V5: now also IC6P.V-, IC7P.V-; no longer IC1P.V-, IC2P.V-
- net AQA: now also IC6A.OUT; no longer IC1A.OUT
- net AQB: now also IC6D.OUT; no longer IC1D.OUT
- net AQC: now also IC6C.OUT; no longer IC1C.OUT
- net AQD: now also IC6B.OUT; no longer IC1B.OUT
- net AQE: now also IC7A.OUT; no longer IC2A.OUT
- net AQF: now also IC7D.OUT; no longer IC2D.OUT
- net AQG: now also IC7C.OUT; no longer IC2C.OUT
- net AQH: now also IC7B.OUT; no longer IC2B.OUT
- net N$15: now also IC6A.IN+; no longer IC1A.+IN
- net N$16: now also IC6B.IN-; no longer IC1B.-IN
- net N$18: now also IC6C.IN+; no longer IC1C.+IN
- net N$19: now also IC6C.IN-; no longer IC1C.-IN
- net N$21: now also IC6A.IN-; no longer IC1A.-IN
- net N$22: now also IC6D.IN+; no longer IC1D.+IN
- net N$23: now also IC6D.IN-; no longer IC1D.-IN
- net N$24: now also IC7A.IN+; no longer IC2A.+IN
- net N$25: now also IC7D.IN+; no longer IC2D.+IN
- net N$26: now also IC6B.IN+; no longer IC1B.+IN
- net N$28: now also IC7B.IN-; no longer IC2B.-IN
- net N$29: now also IC7C.IN+; no longer IC2C.+IN
- net N$30: now also IC7C.IN-; no longer IC2C.-IN
- net N$32: now also IC7D.IN-; no longer IC2D.-IN
- net N$43: now also IC7A.IN-; no longer IC2A.-IN
